Commit message: Improved the URDF model.

File: jaco_model/urdf/jaco_arm.xacro (robot description, xacro)
@@ -32,24 +32,48 @@
   <property name="joint_1_origin_xyz" value="0 0 0.1535" />
   <property name="joint_1_origin_rpy" value="${J_PI} 0 ${J_PI}" />
+  <property name="joint_1_limit_effort" value="30" />
+  <property name="joint_1_limit_velocity" value="0.83" />
+  <property name="joint_1_limit_lower" value="-3.14159265359" />
+  <property name="joint_1_limit_upper" value="3.14159265359" />
   <property name="joint_2" value="jaco_joint_2" />
   <property name="joint_2_axis_xyz" value="0 0 1" />
   <property name="joint_2_origin_xyz" value="0 0 -0.1185" />
   <property name="joint_2_origin_rpy" value="-${J_PI/2} ${J_PI} 0" />
+  <property name="joint_2_limit_effort" value="30" />
+  <property name="joint_2_limit_velocity" value="0.83" />
+  <property name="joint_2_limit_lower" value="-3.89208423195" />
+  <property name="joint_2_limit_upper" value="0.75049157835" />
   <property name="joint_3" value="jaco_joint_3" />
   <property name="joint_3_axis_xyz" value="0 0 -1" />
   <property name="joint_3_origin_xyz" value="0.41 0 0" />
   <property name="joint_3_origin_rpy" value="${J_PI} 0 ${J_PI/2}" />
+  <property name="joint_3_limit_effort" value="30" />
+  <property name="joint_3_limit_velocity" value="0.83" />
+  <property name="joint_3_limit_lower" value="-4.38077642251" />
+  <property name="joint_3_limit_upper" value="1.23918376892" />
   <property name="joint_4" value="jaco_joint_4" />
   <property name="joint_4_axis_xyz" value="0 0 -1" />
   <property name="joint_4_origin_xyz" value="0.207 0 -0.01125" />
   <property name="joint_4_origin_rpy" value="${J_PI} ${J_PI/2} 0" />
+  <property name="joint_4_limit_effort" value="30" />
+  <property name="joint_4_limit_velocity" value="0.83" />
+  <property name="joint_4_limit_lower" value="-3.14159265359" />
+  <property name="joint_4_limit_upper" value="3.14159265359" />
   <property name="joint_5" value="jaco_joint_5" />
   <property name="joint_5_axis_xyz" value="0 0 -1" />
   <property name="joint_5_origin_xyz" value="0.0343 0 -0.06588" />
   <property name="joint_5_origin_rpy" value="0 -${J_PI/180*55} 0" />
+  <property name="joint_5_limit_effort" value="30" />
+  <property name="joint_5_limit_velocity" value="0.83" />
+  <property name="joint_5_limit_lower" value="-3.14159265359" />
+  <property name="joint_5_limit_upper" value="3.14159265359" />
   <property name="joint_6" value="jaco_joint_6" />
   <property name="joint_6_axis_xyz" value="0 0 -1" />
   <property name="joint_6_origin_xyz" value="0.0343 0 -0.06588" />
   <property name="joint_6_origin_rpy" value="-${J_PI/180*55} 0 ${J_PI/2}" />
+  <property name="joint_6_limit_effort" value="30" />
+  <property name="joint_6_limit_velocity" value="0.83" />
+  <property name="joint_6_limit_lower" value="-1.74532925199" />
+  <property name="joint_6_limit_upper" value="4.53785605519" />
   <property name="joint_finger_1" value="jaco_joint_finger_1" />
   <property name="joint_finger_1_axis_xyz" value="0 0 1" />
@@ -97,4 +121,13 @@
  </joint>
 </xacro:macro>
+<xacro:macro name="jaco_joint_revolute" params="joint_name parent child joint_axis_xyz joint_origin_xyz joint_origin_rpy limit_effort limit_velocity limit_lower limit_upper">
+<joint name="${joint_name}" type="revolute">
+    <parent link="${parent}"/>
+    <child link="${child}"/>
+    <axis xyz="${joint_axis_xyz}"/>
+<origin xyz="${joint_origin_xyz}" rpy="${joint_origin_rpy}"/>
+    <limit effort="${limit_effort}" velocity="${limit_velocity}" lower="${limit_lower}" upper="${limit_upper}" />
+ </joint>
+</xacro:macro>
 <xacro:macro name="jaco_finger_joint" params="joint_name type parent child joint_axis_xyz joint_origin_xyz joint_origin_rpy lower_limit upper_limit">
 <joint name="${joint_name}" type="${type}">
@@ -110,15 +143,15 @@
    <xacro:jaco_joint joint_name="${joint_base}" type="fixed" parent="${parent}" child="${link_base}" joint_axis_xyz="${joint_base_axis_xyz}" joint_origin_xyz="${joint_base_origin_xyz}" joint_origin_rpy="${joint_base_origin_rpy}"/>
    <xacro:jaco_link link_name="${link_1}"/>
-   <xacro:jaco_joint joint_name="${joint_1}" type="continuous" parent="${link_base}" child="${link_1}" joint_axis_xyz="${joint_1_axis_xyz}" joint_origin_xyz="${joint_1_origin_xyz}" joint_origin_rpy="${joint_1_origin_rpy}"/>
+   <xacro:jaco_joint_revolute joint_name="${joint_1}" parent="${link_base}" child="${link_1}" joint_axis_xyz="${joint_1_axis_xyz}" joint_origin_xyz="${joint_1_origin_xyz}" joint_origin_rpy="${joint_1_origin_rpy}" limit_effort="${joint_1_limit_effort}" limit_velocity="${joint_1_limit_velocity}" limit_lower="${joint_1_limit_lower}" limit_upper="${joint_1_limit_upper}"/>
    <xacro:jaco_link link_name="${link_2}"/>
-   <xacro:jaco_joint joint_name="${joint_2}" type="continuous" parent="${link_1}" child="${link_2}" joint_axis_xyz="${joint_2_axis_xyz}" joint_origin_xyz="${joint_2_origin_xyz}" joint_origin_rpy="${joint_2_origin_rpy}"/>
+   <xacro:jaco_joint_revolute joint_name="${joint_2}" parent="${link_1}" child="${link_2}" joint_axis_xyz="${joint_2_axis_xyz}" joint_origin_xyz="${joint_2_origin_xyz}" joint_origin_rpy="${joint_2_origin_rpy}" limit_effort="${joint_2_limit_effort}" limit_velocity="${joint_2_limit_velocity}" limit_lower="${joint_2_limit_lower}" limit_upper="${joint_2_limit_upper}"/>
    <xacro:jaco_link link_name="${link_3}"/>
-   <xacro:jaco_joint joint_name="${joint_3}" type="continuous" parent="${link_2}" child="${link_3}" joint_axis_xyz="${joint_3_axis_xyz}" joint_origin_xyz="${joint_3_origin_xyz}" joint_origin_rpy="${joint_3_origin_rpy}"/>
+   <xacro:jaco_joint_revolute joint_name="${joint_3}" parent="${link_2}" child="${link_3}" joint_axis_xyz="${joint_3_axis_xyz}" joint_origin_xyz="${joint_3_origin_xyz}" joint_origin_rpy="${joint_3_origin_rpy}" limit_effort="${joint_3_limit_effort}" limit_velocity="${joint_3_limit_velocity}" limit_lower="${joint_3_limit_lower}" limit_upper="${joint_3_limit_upper}"/>
    <xacro:jaco_link link_name="${link_4}"/>
-   <xacro:jaco_joint joint_name="${joint_4}" type="continuous" parent="${link_3}" child="${link_4}" joint_axis_xyz="${joint_4_axis_xyz}" joint_origin_xyz="${joint_4_origin_xyz}" joint_origin_rpy="${joint_4_origin_rpy}"/>
+   <xacro:jaco_joint_revolute joint_name="${joint_4}" parent="${link_3}" child="${link_4}" joint_axis_xyz="${joint_4_axis_xyz}" joint_origin_xyz="${joint_4_origin_xyz}" joint_origin_rpy="${joint_4_origin_rpy}" limit_effort="${joint_4_limit_effort}" limit_velocity="${joint_4_limit_velocity}" limit_lower="${joint_4_limit_lower}" limit_upper="${joint_4_limit_upper}"/>
    <xacro:jaco_link link_name="${link_5}"/>
-   <xacro:jaco_joint joint_name="${joint_5}" type="continuous" parent="${link_4}" child="${link_5}" joint_axis_xyz="${joint_5_axis_xyz}" joint_origin_xyz="${joint_5_origin_xyz}" joint_origin_rpy="${joint_5_origin_rpy}"/>
+   <xacro:jaco_joint_revolute joint_name="${joint_5}" parent="${link_4}" child="${link_5}" joint_axis_xyz="${joint_5_axis_xyz}" joint_origin_xyz="${joint_5_origin_xyz}" joint_origin_rpy="${joint_5_origin_rpy}" limit_effort="${joint_5_limit_effort}" limit_velocity="${joint_5_limit_velocity}" limit_lower="${joint_5_limit_lower}" limit_upper="${joint_5_limit_upper}"/>
    <xacro:jaco_link link_name="${link_hand}"/>
-   <xacro:jaco_joint joint_name="${joint_6}" type="continuous" parent="${link_5}" child="${link_hand}" joint_axis_xyz="${joint_6_axis_xyz}" joint_origin_xyz="${joint_6_origin_xyz}" joint_origin_rpy="${joint_6_origin_rpy}"/>
+   <xacro:jaco_joint_revolute joint_name="${joint_6}" parent="${link_5}" child="${link_hand}" joint_axis_xyz="${joint_6_axis_xyz}" joint_origin_xyz="${joint_6_origin_xyz}" joint_origin_rpy="${joint_6_origin_rpy}" limit_effort="${joint_6_limit_effort}" limit_velocity="${joint_6_limit_velocity}" limit_lower="${joint_6_limit_lower}" limit_upper="${joint_6_limit_upper}"/>
    <xacro:jaco_link link_name="${link_finger_1}"/>
    <xacro:jaco_finger_joint joint_name="${joint_finger_1}" type="revolute" parent="${link_hand}" child="${link_finger_1}" joint_axis_xyz="${joint_finger_1_axis_xyz}" joint_origin_xyz="${joint_finger_1_origin_xyz}" joint_origin_rpy="${joint_finger_1_origin_rpy}" lower_limit="${joint_finger_1_lower_limit}" upper_limit="${joint_finger_1_upper_limit}"/>

File: jaco_model/urdf/standalone_arm.xacro (robot description, xacro)
@@ -14,5 +14,5 @@
 	xmlns:xacro="http://ros.org/wiki/xacro" name="jaco">
   <xacro:include filename="$(find jaco_model)/urdf/jaco_arm.xacro" />
-<link name="root">
+<link name="jaco_api_origin">
       <visual>
 	<origin xyz="0 0 0" rpy="0 0 0" />
@@ -29,4 +29,4 @@
       </collision>
     </link>
-<xacro:jaco_arm  parent="root"/>
+<xacro:jaco_arm  parent="jaco_api_origin"/>
 </robot>
