Commit message: Standardizing URDF loading and changing continuous joints

File: jaco_model/urdf/standalone_arm.xacro (robot description, xacro)
@@ -14,5 +14,5 @@
 	xmlns:xacro="http://ros.org/wiki/xacro" name="jaco">
   <xacro:include filename="$(find jaco_model)/urdf/jaco_arm.xacro" />
-<link name="jaco_api_origin">
+<link name="root">
       <visual>
 	<origin xyz="0 0 0" rpy="0 0 0" />
@@ -29,4 +29,4 @@
       </collision>
     </link>
-<xacro:jaco_arm  parent="jaco_api_origin"/>
+<xacro:jaco_arm  parent="root"/>
 </robot>
