Commit message: Moved the whole arm moveit stuff to a separate /jaco namespace.

File: jaco_model/urdf/jaco_common.xacro (robot description, xacro)
@@ -53,5 +53,5 @@
     <xacro:macro name="jaco_struct" params="parent basename">
         <xacro:jaco_link link_name="${link_base}"/>
-        <xacro:jaco_joint joint_name="${joint_base}" type="fixed" parent="${parent}" child="${link_base}" joint_axis_xyz="${joint_base_axis_xyz}" joint_origin_xyz="${joint_base_origin_xyz}" joint_origin_rpy="${joint_base_origin_rpy}" joint_lower_limit="0" joint_upper_limit="0"/>
+        <!--xacro:jaco_joint joint_name="${joint_base}" type="fixed" parent="${parent}" child="${link_base}" joint_axis_xyz="${joint_base_axis_xyz}" joint_origin_xyz="${joint_base_origin_xyz}" joint_origin_rpy="${joint_base_origin_rpy}" joint_lower_limit="0" joint_upper_limit="0"/-->
         <xacro:jaco_link link_name="${link_1}"/>
         <xacro:jaco_joint joint_name="${joint_1}" type="continuous" parent="${link_base}" child="${link_1}" joint_axis_xyz="${joint_1_axis_xyz}" joint_origin_xyz="${joint_1_origin_xyz}" joint_origin_rpy="${joint_1_origin_rpy}" joint_lower_limit="${joint_1_lower_limit}" joint_upper_limit="${joint_1_upper_limit}"/>
@@ -71,18 +71,4 @@
          <origin xyz="0 0 ${api_offset}" rpy="0 0 0" />
        </joint>
-       <link name="${api_origin}">
-         <!--
-         <visual>
-           <geometry>
-             <box xyz="0 0 0" size="0.1 0.1 0.1"/>
-           </geometry>
-         </visual>
-         <collision>
-           <geometry>
-             <box xyz="0 0 0" size="0.1 0.1 0.1"/>
-           </geometry>
-         </collision>
-         -->
-        </link>
         <joint name="${link_hand}_to_end_effector" type="fixed">
           <parent link="${link_hand}"/>

Commit message: Added primitive collision elements to Jaco arm.

File: jaco_model/urdf/jaco_common.xacro (robot description, xacro)
@@ -14,5 +14,5 @@
 	xmlns:xacro="http://ros.org/wiki/xacro">
     <property name="J_PI" value="3.1415926535897931" />
-    <xacro:macro name="jaco_link" params="link_name">
+    <xacro:macro name="jaco_link" params="link_name **link_data">
     <link name="${link_name}">
           <visual>
@@ -25,4 +25,9 @@
                     </material>
             </visual>
+            <xacro:insert_block name="link_data" />
+    </link>
+    </xacro:macro>
+    <xacro:macro name="default_link_data" params="link_name">
+         <link_data>
             <collision>
                     <geometry>
@@ -31,5 +36,5 @@
                     </geometry>
             </collision>
-    </link>
+        </link_data>
     </xacro:macro>
     <xacro:macro name="jaco_joint" params="joint_name type parent child joint_axis_xyz joint_origin_xyz joint_origin_rpy joint_lower_limit joint_upper_limit">
@@ -62,17 +67,31 @@
     </xacro:macro>
     <xacro:macro name="jaco_struct" params="parent basename">
-        <xacro:jaco_link link_name="${link_base}"/>
+        <xacro:jaco_link link_name="${link_base}">
+            <xacro:insert_block name="link_base_link_data" />
+        </xacro:jaco_link>
         <!--xacro:jaco_joint joint_name="${joint_base}" type="fixed" parent="${parent}" child="${link_base}" joint_axis_xyz="${joint_base_axis_xyz}" joint_origin_xyz="${joint_base_origin_xyz}" joint_origin_rpy="${joint_base_origin_rpy}" joint_lower_limit="0" joint_upper_limit="0"/-->
-        <xacro:jaco_link link_name="${link_1}"/>
+        <xacro:jaco_link link_name="${link_1}">
+            <xacro:insert_block name="link_1_link_data" />
+        </xacro:jaco_link>
         <xacro:jaco_joint joint_name="${joint_1}" type="continuous" parent="${link_base}" child="${link_1}" joint_axis_xyz="${joint_1_axis_xyz}" joint_origin_xyz="${joint_1_origin_xyz}" joint_origin_rpy="${joint_1_origin_rpy}" joint_lower_limit="${joint_1_lower_limit}" joint_upper_limit="${joint_1_upper_limit}"/>
-        <xacro:jaco_link link_name="${link_2}"/>
+        <xacro:jaco_link link_name="${link_2}">
+            <xacro:insert_block name="link_2_link_data" />
+        </xacro:jaco_link>
         <xacro:jaco_joint joint_name="${joint_2}" type="revolute" parent="${link_1}" child="${link_2}" joint_axis_xyz="${joint_2_axis_xyz}" joint_origin_xyz="${joint_2_origin_xyz}" joint_origin_rpy="${joint_2_origin_rpy}" joint_lower_limit="${joint_2_lower_limit}" joint_upper_limit="${joint_2_upper_limit}"/>
-        <xacro:jaco_link link_name="${link_3}"/>
+        <xacro:jaco_link link_name="${link_3}">
+            <xacro:insert_block name="link_3_link_data" />
+        </xacro:jaco_link>
         <xacro:jaco_joint joint_name="${joint_3}" type="revolute" parent="${link_2}" child="${link_3}" joint_axis_xyz="${joint_3_axis_xyz}" joint_origin_xyz="${joint_3_origin_xyz}" joint_origin_rpy="${joint_3_origin_rpy}" joint_lower_limit="${joint_3_lower_limit}" joint_upper_limit="${joint_3_upper_limit}"/>
-        <xacro:jaco_link link_name="${link_4}"/>
+        <xacro:jaco_link link_name="${link_4}">
+            <xacro:insert_block name="link_4_link_data" />
+        </xacro:jaco_link>
         <xacro:jaco_joint joint_name="${joint_4}" type="continuous" parent="${link_3}" child="${link_4}" joint_axis_xyz="${joint_4_axis_xyz}" joint_origin_xyz="${joint_4_origin_xyz}" joint_origin_rpy="${joint_4_origin_rpy}" joint_lower_limit="${joint_4_lower_limit}" joint_upper_limit="${joint_4_upper_limit}"/>
-        <xacro:jaco_link link_name="${link_5}"/>
+        <xacro:jaco_link link_name="${link_5}">
+            <xacro:insert_block name="link_5_link_data" />
+        </xacro:jaco_link>
         <xacro:jaco_joint joint_name="${joint_5}" type="continuous" parent="${link_4}" child="${link_5}" joint_axis_xyz="${joint_5_axis_xyz}" joint_origin_xyz="${joint_5_origin_xyz}" joint_origin_rpy="${joint_5_origin_rpy}" joint_lower_limit="${joint_5_lower_limit}" joint_upper_limit="${joint_5_upper_limit}"/>
-        <xacro:jaco_link link_name="${link_hand}" />
+        <xacro:jaco_link link_name="${link_hand}">
+            <xacro:insert_block name="link_hand_link_data" />
+        </xacro:jaco_link>
         <xacro:jaco_joint joint_name="${joint_6}" type="continuous" parent="${link_5}" child="${link_hand}" joint_axis_xyz="${joint_6_axis_xyz}" joint_origin_xyz="${joint_6_origin_xyz}" joint_origin_rpy="${joint_6_origin_rpy}" joint_lower_limit="${joint_6_lower_limit}" joint_upper_limit="${joint_6_upper_limit}"/>
        <joint name="${link_base}_to_api_origin" type="fixed">
